File: pcb/snak/snak.kicad_pcb (KiCad board)
At the start: 2 copper layers, 113.1 x 98 mm, 74 parts

Commit message: kicad to pcb
Parts:
- removed the REF** at (184.7, 93.0)
- removed the REF** at (185.9, 92.2)
- removed the REF** at (180.8, 102.8)
- removed the REF** at (187.2, 91.5)
- removed the REF** at (194.8, 92.2)
- added REF**: VIA-0.6mm, VIA-0.6mm, F.Cu at (184.5, 93.0)
- added REF**: VIA-0.6mm, VIA-0.6mm, F.Cu at (185.8, 92.2)
- added REF**: VIA-0.6mm, VIA-0.6mm, F.Cu at (179.0, 102.8)
- added REF**: VIA-0.6mm, VIA-0.6mm, F.Cu at (187.0, 91.5)
- added REF**: VIA-0.6mm, VIA-0.6mm, F.Cu at (194.7, 92.2)
- moved H3 0.50 mm to (163.0, 58.0)
- moved H4 0.50 mm to (163.0, 92.0)
- moved DISP1 0.15 mm to (192.1, 80.8)
- moved MCU1 0.15 mm to (192.1, 74.5)
Connections:
- D1 pad 1: P16 -> P19
- D10 pad 1: P16 -> P19
- D11 pad 1: P14 -> P20
- D12 pad 1: P15 -> P21
- D13 pad 1: P16 -> P19
- D14 pad 1: P14 -> P20
- D15 pad 1: P15 -> P21
- D16 pad 1: P10 -> P18
- D17 pad 1: P10 -> P18
- D2 pad 1: P14 -> P20
- D3 pad 1: P15 -> P21
- D4 pad 1: P16 -> P19
- D5 pad 1: P14 -> P20
- D6 pad 1: P15 -> P21
- D7 pad 1: P16 -> P19
- D8 pad 1: P14 -> P20
- D9 pad 1: P15 -> P21
Other:
- outline, holes or cut-outs redrawn
