File: 30_xiao/03_pcb/rufous.kicad_pcb (KiCad board)
At the start: 2 copper layers, 209.8 x 99 mm, 32 parts

Commit message: update
Parts:
- moved xiao-ble1 0.56 mm to (164.1, 142.8), turned to -90 degrees
Other:
- net class Default removed

Commit message: test xiao fp
Parts:
- moved xiao-ble1 0.56 mm to (163.7, 142.4)
Other:
- net class Default added: clearance 0.2, trace_width 0.25, via_dia 0.8, via_drill 0.4
