File: 28_nice_nano_view/03_pcb/snak_28.kicad_pcb (KiCad board)
At the start: 2 copper layers, 114 x 102 mm, 156 parts

Commit message: update
Parts:
- removed H10: , mounting_hole
- removed the REF** at (107.8, 78.0)
- removed the REF** at (163.2, 65.7)
- removed the REF** at (163.2, 48.2)
- removed the REF** at (181.8, 58.2)
- removed the REF** at (173.3, 113.3)
- removed the REF** at (191.5, 123.6)
- removed the REF** at (107.8, 60.5)
- removed the REF** at (177.5, 64.2)
- removed the REF** at (92.2, 78.0)
- removed the REF** at (126.2, 82.0)
- removed the REF** at (92.2, 60.5)
- removed the REF** at (110.8, 82.0)
- removed the REF** at (110.8, 64.5)
- removed the REF** at (110.8, 47.0)
- removed the REF** at (129.2, 76.0)
- removed the REF** at (129.2, 58.5)
- removed the REF** at (129.2, 41.0)
- removed the REF** at (147.8, 83.2)
- removed the REF** at (147.8, 65.7)
- removed the REF** at (147.8, 48.2)
- removed the REF** at (126.2, 64.5)
- removed the REF** at (166.2, 58.2)
- removed the REF** at (158.5, 108.5)
- removed the REF** at (178.3, 115.6)
- removed the REF** at (126.2, 47.0)
- removed the REF** at (170.5, 64.2)
- removed the REF** at (144.8, 76.0)
- removed the REF** at (174.0, 66.3)
- removed the REF** at (144.8, 58.5)
- removed the REF** at (144.8, 41.0)
- removed the REF** at (174.0, 65.2)
- removed the REF** at (189.2, 86.5)
- removed the REF** at (198.1, 86.5)
- removed the REF** at (163.2, 83.2)
- removed the REF** at (193.7, 87.4)
- removed the REF** at (189.8, 87.4)
- removed the REF** at (197.5, 87.4)
- removed the REF** at (193.7, 88.5)
- removed the REF** at (194.6, 52.2)
- removed the REF** at (174.0, 54.2)
- removed the REF** at (174.0, 49.1)
- removed the REF** at (182.2, 53.7)
- removed the REF** at (183.2, 53.7)
- added REF**: VIA-0.6mm, VIA-0.6mm, F.Cu at (107.0, 78.0)
- added REF**: VIA-0.6mm, VIA-0.6mm, F.Cu at (162.5, 65.7)
- added REF**: VIA-0.6mm, VIA-0.6mm, F.Cu at (162.5, 48.2)
- added REF**: VIA-0.6mm, VIA-0.6mm, F.Cu at (181.0, 76.5)
- added REF**: VIA-0.6mm, VIA-0.6mm, F.Cu at (172.5, 113.1)
- added REF**: VIA-0.6mm, VIA-0.6mm, F.Cu at (190.9, 123.2)
- added REF**: VIA-0.6mm, VIA-0.6mm, F.Cu at (107.0, 60.5)
- added REF**: VIA-0.6mm, VIA-0.6mm, F.Cu at (177.5, 82.5)
- added REF**: VIA-0.6mm, VIA-0.6mm, F.Cu at (93.0, 78.0)
- added REF**: VIA-0.6mm, VIA-0.6mm, F.Cu at (125.5, 82.0)
- added REF**: VIA-0.6mm, VIA-0.6mm, F.Cu at (93.0, 60.5)
- added REF**: VIA-0.6mm, VIA-0.6mm, F.Cu at (111.5, 82.0)
- added REF**: VIA-0.6mm, VIA-0.6mm, F.Cu at (111.5, 64.5)
- added REF**: VIA-0.6mm, VIA-0.6mm, F.Cu at (111.5, 47.0)
- added REF**: VIA-0.6mm, VIA-0.6mm, F.Cu at (130.0, 76.0)
- added REF**: VIA-0.6mm, VIA-0.6mm, F.Cu at (130.0, 58.5)
- added REF**: VIA-0.6mm, VIA-0.6mm, F.Cu at (130.0, 41.0)
- added REF**: VIA-0.6mm, VIA-0.6mm, F.Cu at (148.5, 83.2)
- added REF**: VIA-0.6mm, VIA-0.6mm, F.Cu at (148.5, 65.7)
- added REF**: VIA-0.6mm, VIA-0.6mm, F.Cu at (148.5, 48.2)
- added REF**: VIA-0.6mm, VIA-0.6mm, F.Cu at (125.5, 64.5)
- added REF**: VIA-0.6mm, VIA-0.6mm, F.Cu at (167.0, 76.5)
- added REF**: VIA-0.6mm, VIA-0.6mm, F.Cu at (159.2, 108.8)
- added REF**: VIA-0.6mm, VIA-0.6mm, F.Cu at (178.9, 116.0)
- added REF**: VIA-0.6mm, VIA-0.6mm, F.Cu at (125.5, 47.0)
- added REF**: VIA-0.6mm, VIA-0.6mm, F.Cu at (170.5, 82.5)
- added REF**: VIA-0.6mm, VIA-0.6mm, F.Cu at (144.0, 76.0)
- added REF**: VIA-0.6mm, VIA-0.6mm, F.Cu at (174.0, 84.6)
- added REF**: VIA-0.6mm, VIA-0.6mm, F.Cu at (144.0, 58.5)
- added REF**: VIA-0.6mm, VIA-0.6mm, F.Cu at (144.0, 41.0)
- added REF**: VIA-0.6mm, VIA-0.6mm, F.Cu at (174.0, 83.5)
- added REF**: VIA-0.6mm, VIA-0.6mm, F.Cu at (189.2, 86.8)
- added REF**: VIA-0.6mm, VIA-0.6mm, F.Cu at (198.1, 86.8)
- added REF**: VIA-0.6mm, VIA-0.6mm, F.Cu at (162.5, 83.2)
- added REF**: VIA-0.6mm, VIA-0.6mm, F.Cu at (193.7, 87.7)
- added REF**: VIA-0.6mm, VIA-0.6mm, F.Cu at (189.8, 87.7)
- added REF**: VIA-0.6mm, VIA-0.6mm, F.Cu at (197.5, 87.7)
- added REF**: VIA-0.6mm, VIA-0.6mm, F.Cu at (193.7, 88.8)
- added REF**: VIA-0.6mm, VIA-0.6mm, F.Cu at (194.6, 52.5)
- added REF**: VIA-0.6mm, VIA-0.6mm, F.Cu at (195.2, 96.8)
- added REF**: VIA-0.6mm, VIA-0.6mm, F.Cu at (200.2, 96.8)
- added REF**: VIA-0.6mm, VIA-0.6mm, F.Cu at (183.2, 52.9)
- added REF**: VIA-0.6mm, VIA-0.6mm, F.Cu at (183.2, 54.0)
- DISP1: footprint nice!view -> ceoloide:nice_view
- moved H9 79.1 mm to (201.2, 54.0), turned to 0 degrees
- moved JST1 52.5 mm to (198.8, 96.8), turned to 270 degrees
- moved H7 39.8 mm to (171.0, 91.7)
- moved H8 36.1 mm to (170.4, 126.9), turned to -18 degrees
- moved TP1 21.2 mm to (171.0, 61.9)
- moved D12 18.3 mm to (181.5, 79.5)
- moved D26 18.3 mm to (166.5, 79.5)
- moved S12 18.3 mm to (174.0, 81.0)
- moved H1 2.00 mm to (104.5, 54.4)
- moved H2 2.00 mm to (104.5, 93.2)
- moved H3 1.80 mm to (118.5, 42.1)
- moved H5 1.80 mm to (155.5, 43.4)
- moved D28 0.75 mm to (176.9, 118.3)
- moved D27 0.75 mm to (157.8, 111.5)
- moved D1 0.75 mm to (107.5, 81.0)
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Connections:
- net inner_top renamed inner_mid
- D12 pad 1: R1 -> R2
- D26 pad 1: R1 -> R2
- DISP1 pad 14: MOSI -> CS
- DISP1 pad 15: SCK -> GND
- DISP1 pad 16: GND -> SCK
- DISP1 pad 17: CS -> MOSI
- DISP1 pad 24: MOSI -> CS
- DISP1 pad 25: SCK -> GND
- DISP1 pad 26: GND -> SCK
- DISP1 pad 27: CS -> MOSI
Routing:
- net SCK: track 0.00 -> 3.50 mm
- net MOSI: track 0.00 -> 3.50 mm
- net GND: track 0.00 -> 3.50 mm
- net CS: track 0.00 -> 3.50 mm
Other:
- outline, holes or cut-outs redrawn

Commit message: add scrollwheel to 28 key config
Parts:
- removed the REF** at (194.6, 52.5)
- removed the REF** at (183.2, 52.9)
- removed the REF** at (183.2, 54.0)
- added REF**: VIA-0.6mm, VIA-0.6mm, F.Cu at (193.7, 52.5)
- added REF**: VIA-0.6mm, VIA-0.6mm, F.Cu at (178.4, 48.2)
- added REF**: VIA-0.6mm, VIA-0.6mm, F.Cu at (177.6, 49.1)
- added REF**: RollerEncoder_Panasonic_EVQWGD001, RollerEncoder_Panasonic_EVQWGD001, F.Cu at (174.5, 61.1)
- moved SW2 6.49 mm to (180.6, 50.8), turned to 51 degrees
- moved TP1 3.00 mm to (174.0, 61.9)
- moved SW1 0.90 mm to (193.7, 53.6)
Connections:
- MCU1 pad 123: F1 -> SW1
- MCU1 pad 124: F2 -> SW2

Commit message: update scrollwheel rotation and placement
Parts:
- removed the REF** at (172.5, 113.1)
- removed the REF** at (190.9, 123.2)
- removed the REF** at (167.4, 117.7)
- removed the REF** at (184.8, 126.5)
- removed the REF** at (159.2, 108.8)
- removed the REF** at (178.9, 116.0)
- removed the REF** at (160.7, 115.5)
- removed the REF** at (178.8, 122.9)
- removed the REF** at (163.4, 118.6)
- removed the REF** at (180.7, 126.5)
- removed the REF** at (163.7, 117.6)
- removed the REF** at (181.3, 125.6)
- removed the REF** at (176.2, 113.0)
- removed the REF** at (159.0, 104.5)
- removed the REF** at (179.7, 111.8)
- removed the REF** at (193.7, 52.5)
- removed the REF** at (178.4, 48.2)
- removed the REF** at (177.6, 49.1)
- added REF**: VIA-0.6mm, VIA-0.6mm, F.Cu at (172.5, 110.6)
- added REF**: VIA-0.6mm, VIA-0.6mm, F.Cu at (190.9, 120.7)
- added REF**: VIA-0.6mm, VIA-0.6mm, F.Cu at (167.4, 115.2)
- added REF**: VIA-0.6mm, VIA-0.6mm, F.Cu at (184.8, 124.0)
- added REF**: VIA-0.6mm, VIA-0.6mm, F.Cu at (159.2, 106.3)
- added REF**: VIA-0.6mm, VIA-0.6mm, F.Cu at (178.9, 113.5)
- added REF**: VIA-0.6mm, VIA-0.6mm, F.Cu at (160.7, 113.0)
- added REF**: VIA-0.6mm, VIA-0.6mm, F.Cu at (178.8, 120.4)
- added REF**: VIA-0.6mm, VIA-0.6mm, F.Cu at (163.4, 116.1)
- added REF**: VIA-0.6mm, VIA-0.6mm, F.Cu at (180.7, 124.0)
- added REF**: VIA-0.6mm, VIA-0.6mm, F.Cu at (163.7, 115.1)
- added REF**: VIA-0.6mm, VIA-0.6mm, F.Cu at (181.3, 123.1)
- added REF**: VIA-0.6mm, VIA-0.6mm, F.Cu at (176.2, 110.5)
- added REF**: VIA-0.6mm, VIA-0.6mm, F.Cu at (159.0, 102.0)
- added REF**: VIA-0.6mm, VIA-0.6mm, F.Cu at (179.7, 109.3)
- added REF**: VIA-0.6mm, VIA-0.6mm, F.Cu at (193.7, 52.5)
- added REF**: VIA-0.6mm, VIA-0.6mm, F.Cu at (171.5, 43.9)
- added REF**: VIA-0.6mm, VIA-0.6mm, F.Cu at (170.8, 44.9)
- moved SW2 8.02 mm to (174.0, 46.2), turned to 58 degrees
- moved D13 2.50 mm to (172.1, 113.6)
- moved D14 2.50 mm to (189.8, 123.5)
- moved D27 2.50 mm to (157.8, 109.0)
- moved D28 2.50 mm to (176.9, 115.8)
- moved H8 2.50 mm to (170.4, 124.4)
- moved S13 2.50 mm to (164.5, 112.7)
- moved S14 2.50 mm to (182.6, 120.9)
- moved REF** 1.14 mm to (174.5, 62.2)
Connections:
- MCU1 pad 123: SW1 -> SW2
- MCU1 pad 124: SW2 -> SW1
Other:
- board size 114 x 102 mm -> 114 x 99.6 mm

Commit message: update 28
Parts:
- removed the REF** at (189.2, 86.8)
- removed the REF** at (198.1, 86.8)
- removed the REF** at (193.7, 87.7)
- removed the REF** at (189.8, 87.7)
- removed the REF** at (197.5, 87.7)
- removed the REF** at (193.7, 88.8)
- removed the REF** at (193.7, 52.5)
- removed the REF** at (195.2, 96.8)
- removed the REF** at (200.2, 96.8)
- removed the REF** at (171.5, 43.9)
- removed the REF** at (170.8, 44.9)
- added REF**: VIA-0.6mm, VIA-0.6mm, F.Cu at (190.0, 86.8)
- added REF**: VIA-0.6mm, VIA-0.6mm, F.Cu at (198.8, 86.8)
- added REF**: VIA-0.6mm, VIA-0.6mm, F.Cu at (194.4, 87.7)
- added REF**: VIA-0.6mm, VIA-0.6mm, F.Cu at (190.6, 87.7)
- added REF**: VIA-0.6mm, VIA-0.6mm, F.Cu at (198.2, 87.7)
- added REF**: VIA-0.6mm, VIA-0.6mm, F.Cu at (194.4, 88.8)
- added REF**: VIA-0.6mm, VIA-0.6mm, F.Cu at (194.4, 52.5)
- added REF**: VIA-0.6mm, VIA-0.6mm, F.Cu at (195.9, 96.8)
- added REF**: VIA-0.6mm, VIA-0.6mm, F.Cu at (200.9, 96.8)
- added REF**: VIA-0.6mm, VIA-0.6mm, F.Cu at (177.7, 47.8)
- added REF**: VIA-0.6mm, VIA-0.6mm, F.Cu at (177.0, 48.8)
- moved SW2 7.30 mm to (180.0, 50.4), turned to 52 degrees
- moved H2 2.46 mm to (106.8, 92.2)
- moved H1 2.25 mm to (106.8, 54.4)
- moved H7 1.50 mm to (172.5, 91.7)
- moved H5 1.25 mm to (155.5, 42.1)
- moved TP1 1.25 mm to (172.8, 61.8)
- moved H6 0.80 mm to (155.5, 98.0)
- moved DISP1 0.75 mm to (194.4, 74.3)
- moved H9 0.75 mm to (201.9, 54.0)
- moved JST1 0.75 mm to (199.6, 96.8)
- moved MCU1 0.75 mm to (194.4, 70.2)
- moved REF** 0.75 mm to (175.2, 62.2)
- moved SW1 0.75 mm to (194.4, 53.6)
- moved H4 0.25 mm to (118.5, 97.4)
Other:
- board size 114 x 99.6 mm -> 114.8 x 99.6 mm

Commit message: update 28 config
Parts:
- moved REF** 1.77 mm to (174.0, 63.5)
- moved H4 0.65 mm to (118.5, 98.0)
Changed lines of the file:
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@@
             )
             (module mounting_hole (layer F.Cu)
-                (at 118.5 97.4 0)
+                (at 118.5 98.05 0)
                 (fp_text reference "H4" (at 0 3) (layer F.SilkS) hide
                     (effects (font (size 1 1) (thickness 0.15)))
@@
       )
         (module RollerEncoder_Panasonic_EVQWGD001 (layer F.Cu)
-        (at 175.25 62.245 180)
+        (at 174 63.5 180)
         (fp_text reference REF** (at 0 0 180) (layer F.Fab) (effects (font (size 1 1) (thickness 0.15))))
         (fp_text value RollerEncoder_Panasonic_EVQWGD001 (at -0.1 9 180) (layer F.Fab) (effects (font (size 1 1) (thickness 0.15))))
@@
 (gr_circle (center 106.75 92.15) (end 107.75 92.15) (layer Eco1.User) (width 0.15))
 (gr_circle (center 118.5 42.1) (end 119.5 42.1) (layer Eco1.User) (width 0.15))
-(gr_circle (center 118.5 97.4) (end 119.5 97.4) (layer Eco1.User) (width 0.15))
+(gr_circle (center 118.5 98.05) (end 119.5 98.05) (layer Eco1.User) (width 0.15))
 (gr_circle (center 155.5 42.1) (end 156.5 42.1) (layer Eco1.User) (width 0.15))
 (gr_circle (center 155.5 98.05) (end 156.5 98.05) (layer Eco1.User) (width 0.15))
@@
 (gr_circle (center 170.43886559999999 124.35568) (end 171.43886559999999 124.35568) (layer Eco1.User) (width 0.15))
 (gr_circle (center 201.925 53.975) (end 202.925 53.975) (layer Eco1.User) (width 0.15))
+(gr_circle (center 172.75 52.32) (end 173.75 52.32) (layer Eco1.User) (width 0.15))
+(gr_circle (center 172.75 71.32) (end 173.75 71.32) (layer Eco1.User) (width 0.15))
 (gr_line (start 93.05 89.45) (end 106.95 89.45) (angle 90) (layer Eco1.User) (width 0.15))
 (gr_line (start 106.95 89.45) (end 106.95 75.55) (angle 90) (layer Eco1.User) (width 0.15))
@@
 (gr_circle (center 106.75 92.15) (end 108.25 92.15) (layer Eco2.User) (width 0.15))
 (gr_circle (center 118.5 42.1) (end 120 42.1) (layer Eco2.User) (width 0.15))
-(gr_circle (center 118.5 97.4) (end 120 97.4) (layer Eco2.User) (width 0.15))
+(gr_circle (center 118.5 98.05) (end 120 98.05) (layer Eco2.User) (width 0.15))
 (gr_circle (center 155.5 42.1) (end 157 42.1) (layer Eco2.User) (width 0.15))
 (gr_circle (center 155.5 98.05) (end 157 98.05) (layer Eco2.User) (width 0.15))
@@
 (gr_circle (center 170.43886559999999 124.35568) (end 171.93886559999999 124.35568) (layer Eco2.User) (width 0.15))
 (gr_circle (center 201.925 53.975) (end 203.425 53.975) (layer Eco2.User) (width 0.15))
+(gr_circle (center 172.75 52.32) (end 174.25 52.32) (layer Eco2.User) (width 0.15))
+(gr_circle (center 172.75 71.32) (end 174.25 71.32) (layer Eco2.User) (width 0.15))
 )
