File: 28_nice_nano_view/03_pcb/snak_28.kicad_pcb (KiCad board)
At the start: 2 copper layers, 114.8 x 99.6 mm, 172 parts

Commit message: add cli config
Parts:
- MCU1: footprint ceoloide:nice_nano -> ceoloide:mcu_nice_nano
- moved TP1 1.25 mm to (172.8, 62.4), turned to 0 degrees
Connections:
- MCU1 pad 1: RAW -> MCU1_1
- MCU1 pad 10: SW1 -> MCU1_10
- MCU1 pad 11: SW2 -> MCU1_11
- MCU1 pad 113: R4 -> F2
- MCU1 pad 114: CS -> SW2
- MCU1 pad 115: SCK -> SW1
- MCU1 pad 116: MOSI -> C5
- MCU1 pad 117: R3 -> C4
- MCU1 pad 118: R2 -> C3
- MCU1 pad 119: R1 -> C2
- MCU1 pad 12: F2 -> MCU1_12
- MCU1 pad 120: F1 -> C1
- MCU1 pad 121: GND -> VCC
- MCU1 pad 122: GND -> RST
- MCU1 pad 123: TPD -> GND
- MCU1 pad 124: TPC -> RAW
- MCU1 pad 2: GND -> MCU1_2
- MCU1 pad 3: RST -> MCU1_3
- MCU1 pad 4: VCC -> MCU1_4
- MCU1 pad 5: C1 -> MCU1_5
- MCU1 pad 6: C2 -> MCU1_6
- MCU1 pad 7: C3 -> MCU1_7
- MCU1 pad 8: C4 -> MCU1_8
- MCU1 pad 9: C5 -> MCU1_9
Routing:
- net (no net): track 0.00 -> 333.1 mm
- net R2: track 101.6 -> 0.00 mm
- net pinky_mid: track 101.4 -> 0.00 mm
- net RAW: track 50.9 -> 0.00 mm
- net R4: track 50.9 -> 0.00 mm
- net index_bot: track 14.2 -> 0.00 mm
- net C1: track 14.2 -> 0.00 mm
